File: _saved_linjal.sch (KiCad schematic (older format))
At the start: 26 parts, among them SW1 FSM4JSMAATR, U1 LM555

Commit message: finished schematic. rough drawing of layout
Parts:
- C1: footprint (none) -> Capacitors_SMD:C_0603
- D1, D10, D11, D12, D13, D14, D15, D16, D17, D18, D2, D3, D4, D5, D6, D7, D8, D9: footprint (none) -> LEDs:LED_0603
- R1, R2, R3, R4: footprint (none) -> Resistors_SMD:R_0603
- SW1: footprint (none) -> FSM4JSMAATR:SW_FSM4JSMAATR
- U1: footprint (none) -> digikey-footprints:8-SOIC
Other:
- note added: "Output can source or sink 200mA\n"
Changed lines of the file:
@@
 F 0 "SW1" H 4000 2417 50  0000 C CNN
 F 1 "FSM4JSMAATR" H 4000 2326 50  0000 C CNN
-F 2 "" H 4000 2150 50  0001 C CNN
+F 2 "FSM4JSMAATR:SW_FSM4JSMAATR" H 4000 2150 50  0001 C CNN
 F 3 "http://www.farnell.com/datasheets/2074932.pdf?_ga=2.114085255.1882748413.1533757880-423028813.1532970484" H 4000 2150 50  0001 C CNN
 F 4 "http://no.farnell.com/alcoswitch-te-connectivity/fsm4jsmaatr/tactile-switch-spst-no-0-05a-24v/dp/2610936" H 4000 2150 50  0001 C CNN "Link"
@@
 F 0 "U1" H 5300 3228 50  0000 C CNN
 F 1 "LM555" H 5300 3137 50  0000 C CNN
-F 2 "" H 5300 2650 50  0001 C CNN
+F 2 "digikey-footprints:8-SOIC" H 5300 2650 50  0001 C CNN
 F 3 "http://www.ti.com/lit/ds/symlink/lm555.pdf" H 5300 2650 50  0001 C CNN
 	1    5300 2650
@@
 F 0 "R1" H 4459 2346 50  0000 L CNN
 F 1 "1M" H 4459 2255 50  0000 L CNN
-F 2 "" H 4400 2300 50  0001 C CNN
+F 2 "Resistors_SMD:R_0603" H 4400 2300 50  0001 C CNN
 F 3 "~" H 4400 2300 50  0001 C CNN
 	1    4400 2300
@@
 F 0 "C1" H 5892 3296 50  0000 L CNN
 F 1 "300n" H 5892 3205 50  0000 L CNN
-F 2 "" H 5800 3250 50  0001 C CNN
+F 2 "Capacitors_SMD:C_0603" H 5800 3250 50  0001 C CNN
 F 3 "~" H 5800 3250 50  0001 C CNN
 	1    5800 3250
@@
 F 0 "R2" V 5104 1900 50  0000 C CNN
 F 1 "20k" V 5195 1900 50  0000 C CNN
-F 2 "" H 5300 1900 50  0001 C CNN
+F 2 "Resistors_SMD:R_0603" H 5300 1900 50  0001 C CNN
 F 3 "~" H 5300 1900 50  0001 C CNN
 	1    5300 1900
@@
 F 0 "D2" V 6496 2482 50  0000 R CNN
 F 1 "LED" V 6405 2482 50  0000 R CNN
-F 2 "" V 6450 2550 50  0001 C CNN
+F 2 "LEDs:LED_0603" V 6450 2550 50  0001 C CNN
 F 3 "~" V 6450 2550 50  0001 C CNN
 	1    6450 2550
@@
 F 0 "D3" V 6796 2482 50  0000 R CNN
 F 1 "LED" V 6705 2482 50  0000 R CNN
-F 2 "" V 6750 2550 50  0001 C CNN
+F 2 "LEDs:LED_0603" V 6750 2550 50  0001 C CNN
 F 3 "~" V 6750 2550 50  0001 C CNN
 	1    6750 2550
@@
 F 0 "D4" V 7096 2482 50  0000 R CNN
 F 1 "LED" V 7005 2482 50  0000 R CNN
-F 2 "" V 7050 2550 50  0001 C CNN
+F 2 "LEDs:LED_0603" V 7050 2550 50  0001 C CNN
 F 3 "~" V 7050 2550 50  0001 C CNN
 	1    7050 2550
@@
 F 0 "D5" V 7396 2482 50  0000 R CNN
 F 1 "LED" V 7305 2482 50  0000 R CNN
-F 2 "" V 7350 2550 50  0001 C CNN
+F 2 "LEDs:LED_0603" V 7350 2550 50  0001 C CNN
 F 3 "~" V 7350 2550 50  0001 C CNN
 	1    7350 2550
@@
 F 0 "D6" V 7696 2482 50  0000 R CNN
 F 1 "LED" V 7605 2482 50  0000 R CNN
-F 2 "" V 7650 2550 50  0001 C CNN
+F 2 "LEDs:LED_0603" V 7650 2550 50  0001 C CNN
 F 3 "~" V 7650 2550 50  0001 C CNN
 	1    7650 2550
@@
 F 0 "D7" V 7996 2482 50  0000 R CNN
 F 1 "LED" V 7905 2482 50  0000 R CNN
-F 2 "" V 7950 2550 50  0001 C CNN
+F 2 "LEDs:LED_0603" V 7950 2550 50  0001 C CNN
 F 3 "~" V 7950 2550 50  0001 C CNN
 	1    7950 2550
@@
 F 0 "D8" V 8296 2482 50  0000 R CNN
 F 1 "LED" V 8205 2482 50  0000 R CNN
-F 2 "" V 8250 2550 50  0001 C CNN
+F 2 "LEDs:LED_0603" V 8250 2550 50  0001 C CNN
 F 3 "~" V 8250 2550 50  0001 C CNN
 	1    8250 2550
@@
 F 0 "D9" V 8596 2482 50  0000 R CNN
 F 1 "LED" V 8505 2482 50  0000 R CNN
-F 2 "" V 8550 2550 50  0001 C CNN
+F 2 "LEDs:LED_0603" V 8550 2550 50  0001 C CNN
 F 3 "~" V 8550 2550 50  0001 C CNN
 	1    8550 2550
@@
 F 0 "D10" V 8896 2482 50  0000 R CNN
 F 1 "LED" V 8805 2482 50  0000 R CNN
-F 2 "" V 8850 2550 50  0001 C CNN
+F 2 "LEDs:LED_0603" V 8850 2550 50  0001 C CNN
 F 3 "~" V 8850 2550 50  0001 C CNN
 	1    8850 2550
@@
 F 0 "D11" V 9196 2482 50  0000 R CNN
 F 1 "LED" V 9105 2482 50  0000 R CNN
-F 2 "" V 9150 2550 50  0001 C CNN
+F 2 "LEDs:LED_0603" V 9150 2550 50  0001 C CNN
 F 3 "~" V 9150 2550 50  0001 C CNN
 	1    9150 2550
@@
 F 0 "D12" V 9496 2482 50  0000 R CNN
 F 1 "LED" V 9405 2482 50  0000 R CNN
-F 2 "" V 9450 2550 50  0001 C CNN
+F 2 "LEDs:LED_0603" V 9450 2550 50  0001 C CNN
 F 3 "~" V 9450 2550 50  0001 C CNN
 	1    9450 2550
@@
 F 0 "D13" V 9796 2482 50  0000 R CNN
 F 1 "LED" V 9705 2482 50  0000 R CNN
-F 2 "" V 9750 2550 50  0001 C CNN
+F 2 "LEDs:LED_0603" V 9750 2550 50  0001 C CNN
 F 3 "~" V 9750 2550 50  0001 C CNN
 	1    9750 2550
@@
 F 0 "D14" V 10096 2482 50  0000 R CNN
 F 1 "LED" V 10005 2482 50  0000 R CNN
-F 2 "" V 10050 2550 50  0001 C CNN
+F 2 "LEDs:LED_0603" V 10050 2550 50  0001 C CNN
 F 3 "~" V 10050 2550 50  0001 C CNN
 	1    10050 2550
@@
 F 0 "D15" V 10396 2482 50  0000 R CNN
 F 1 "LED" V 10305 2482 50  0000 R CNN
-F 2 "" V 10350 2550 50  0001 C CNN
+F 2 "LEDs:LED_0603" V 10350 2550 50  0001 C CNN
 F 3 "~" V 10350 2550 50  0001 C CNN
 	1    10350 2550
@@
 F 0 "D16" V 10696 2482 50  0000 R CNN
 F 1 "LED" V 10605 2482 50  0000 R CNN
-F 2 "" V 10650 2550 50  0001 C CNN
+F 2 "LEDs:LED_0603" V 10650 2550 50  0001 C CNN
 F 3 "~" V 10650 2550 50  0001 C CNN
 	1    10650 2550
@@
 F 0 "D17" V 10996 2482 50  0000 R CNN
 F 1 "LED" V 10905 2482 50  0000 R CNN
-F 2 "" V 10950 2550 50  0001 C CNN
+F 2 "LEDs:LED_0603" V 10950 2550 50  0001 C CNN
 F 3 "~" V 10950 2550 50  0001 C CNN
 	1    10950 2550
@@
 F 0 "D1" V 6196 2482 50  0000 R CNN
 F 1 "LED" V 6105 2482 50  0000 R CNN
-F 2 "" V 6150 2550 50  0001 C CNN
+F 2 "LEDs:LED_0603" V 6150 2550 50  0001 C CNN
 F 3 "~" V 6150 2550 50  0001 C CNN
 	1    6150 2550
@@
 F 0 "D18" V 11296 2482 50  0000 R CNN
 F 1 "LED" V 11205 2482 50  0000 R CNN
-F 2 "" V 11250 2550 50  0001 C CNN
+F 2 "LEDs:LED_0603" V 11250 2550 50  0001 C CNN
 F 3 "~" V 11250 2550 50  0001 C CNN
 	1    11250 2550
@@
 F 0 "R4" V 8754 2900 50  0000 C CNN
 F 1 "10R" V 8845 2900 50  0000 C CNN
-F 2 "" H 8950 2900 50  0001 C CNN
+F 2 "Resistors_SMD:R_0603" H 8950 2900 50  0001 C CNN
 F 3 "~" H 8950 2900 50  0001 C CNN
 	1    8950 2900
@@
 F 0 "R3" V 8454 2900 50  0000 C CNN
 F 1 "10R" V 8545 2900 50  0000 C CNN
-F 2 "" H 8650 2900 50  0001 C CNN
+F 2 "Resistors_SMD:R_0603" H 8650 2900 50  0001 C CNN
 F 3 "~" H 8650 2900 50  0001 C CNN
 	1    8650 2900
@@
 Wire Wire Line
 	8650 2650 8850 2650
+Text Notes 6000 2400 0    50   ~ 0
+Output can source or sink 200mA\n
 $EndSCHEMATC
