File: linjal.kicad_pcb (KiCad board)
At the start: 2 copper layers, 210 x 35 mm, 0 parts

Commit message: finished schematic. rough drawing of layout
Parts:
- added BT1: BC-2001, footprints:BC-2001, B.Cu at (70.4, 80.8)
- added C1: 300n, Capacitors_SMD:C_0603, B.Cu at (113.3, 87.3)
- added D1: LED, LEDs:LED_0603, B.Cu at (238.0, 77.5)
- added D10: LED, LEDs:LED_0603, B.Cu at (251.1, 73.1)
- added D11: LED, LEDs:LED_0603, B.Cu at (252.8, 81.5)
- added D12: LED, LEDs:LED_0603, B.Cu at (247.4, 72.1)
- added D13: LED, LEDs:LED_0603, B.Cu at (239.7, 85.9)
- added D14: LED, LEDs:LED_0603, B.Cu at (239.0, 73.8)
- added D15: LED, LEDs:LED_0603, B.Cu at (243.4, 86.9)
- added D16: LED, LEDs:LED_0603, B.Cu at (250.1, 76.8)
- added D17: LED, LEDs:LED_0603, B.Cu at (253.7, 77.8)
- added D18: LED, LEDs:LED_0603, B.Cu at (251.8, 85.1)
- added D2: LED, LEDs:LED_0603, B.Cu at (248.1, 84.2)
- added D3: LED, LEDs:LED_0603, B.Cu at (243.7, 71.1)
- added D4: LED, LEDs:LED_0603, B.Cu at (245.4, 79.5)
- added D5: LED, LEDs:LED_0603, B.Cu at (247.1, 87.8)
- added D6: LED, LEDs:LED_0603, B.Cu at (249.1, 80.5)
- added D7: LED, LEDs:LED_0603, B.Cu at (241.7, 78.5)
- added D8: LED, LEDs:LED_0603, B.Cu at (236.1, 84.9)
- added D9: LED, LEDs:LED_0603, B.Cu at (242.7, 74.8)
- added R1: 1M, Resistors_SMD:R_0603, B.Cu at (110.5, 75.6)
- added R2: 20k, Resistors_SMD:R_0603, B.Cu at (109.7, 87.3)
- added R3: 10R, Resistors_SMD:R_0603, B.Cu at (251.1, 91.3)
- added R4: 10R, Resistors_SMD:R_0603, B.Cu at (254.1, 91.4)
- added SW1: FSM4JSMAATR, FSM4JSMAATR:SW_FSM4JSMAATR, B.Cu at (96.5, 80.5)
- added U1: LM555, digikey-footprints:8-SOIC, B.Cu at (109.8, 80.6)
Routing:
- net Net-(D1-Pad1): track 0.00 -> 98.7 mm
- net Net-(D1-Pad2): track 0.00 -> 97.0 mm
- net Net-(BT1-Pad1): track 0.00 -> 38.9 mm
- net Net-(R1-Pad1): track 0.00 -> 16.3 mm
- net Net-(C1-Pad1): track 0.00 -> 14.5 mm, vias 0 -> 2
- net GND: track 0.00 -> 8.24 mm, vias 0 -> 2
- added copper zone on F.Cu, net GND
- added copper zone on B.Cu, net Net-(D1-Pad2)

Commit message: added some footprints
Parts:
- added 0201: R_0201, Resistors_SMD:R_0201, F.Cu at (62.4, 89.1)
- added 0402: R_0402, Resistors_SMD:R_0402, F.Cu at (64.2, 89.1)
- added 0604: R_0603, Resistors_SMD:R_0603, F.Cu at (66.3, 89.1)
- added 0805: R_0805, Resistors_SMD:R_0805, F.Cu at (68.7, 89.1)
- added M2: MountingHole_2.2mm_M2, Mounting_Holes:MountingHole_2.2mm_M2, B.Cu at (207.8, 88.5)
- added M2: MountingHole_2.2mm_M2, Mounting_Holes:MountingHole_2.2mm_M2, F.Cu at (207.8, 88.5)
- added M3: MountingHole_3.2mm_M3, Mounting_Holes:MountingHole_3.2mm_M3, B.Cu at (55.0, 89.0)
- added M3: MountingHole_3.2mm_M3, Mounting_Holes:MountingHole_3.2mm_M3, B.Cu at (211.4, 88.5)
- added M3: MountingHole_3.2mm_M3, Mounting_Holes:MountingHole_3.2mm_M3, F.Cu at (211.4, 88.5)
- added M4: MountingHole_4.3mm_M4, Mounting_Holes:MountingHole_4.3mm_M4, B.Cu at (216.1, 88.5)
- added M4: MountingHole_4.3mm_M4, Mounting_Holes:MountingHole_4.3mm_M4, F.Cu at (216.1, 88.5)
- added M5: MountingHole_5mm, Mounting_Holes:MountingHole_5mm, B.Cu at (221.7, 88.5)
- added M5: MountingHole_5mm, Mounting_Holes:MountingHole_5mm, F.Cu at (221.7, 88.5)
- added NPN: npn, footprints:npn, F.Cu at (212.8, 75.9)
Routing:
- net Net-(C1-Pad1): track 14.5 -> 22.9 mm, vias 2 -> 0
- net GND: track 8.24 -> 13.1 mm, vias 2 -> 3
- net (no net): vias 0 -> 3
Other:
- net class Default: trace_width 0.25 -> 0.254
- rule trace_min: 0.2 -> 0.0889
- board text added: "0.6 mm"
- board text added: "0.8 mm"
- board text added: "1 mil = 0.0254 mm"
- board text added: "1.0 mm"
- board text added: "10 mil"
- board text added: "5 mil"
- board text added: "6 mil"
- board text added: "8 mil"
- board text added: "SMD resistor sizes (imperial)"
- board text added: "Trace width"

Commit message: BOM
Parts:
- removed NPN: npn, footprints:npn
- added 1.27mm: Pin_Header_Straight_1x02_Pitch1.27mm, Pin_Headers:Pin_Header_Straight_1x02_Pitch1.27mm, F.Cu at (179.1, 89.2)
- added 2.54mm: Pin_Header_Straight_1x02_Pitch2.54mm, Pin_Headers:Pin_Header_Straight_1x02_Pitch2.54mm, F.Cu at (184.2, 88.6)
- added G***: LOGO, footprints:silk_draws_tables, F.Cu at (149.6, 81.5)
- added G***: LOGO, footprints:silk_draws, F.Cu at (99.7, 80.4)
- added SOD-123: SOD-123, digikey-footprints:SOD-123, F.Cu at (196.0, 70.6)
- added SOD-323: SOD-323, digikey-footprints:SOD-323, F.Cu at (196.2, 75.2)
- added SOIC-8: 8-SOIC, digikey-footprints:8-SOIC, F.Cu at (205.5, 72.4)
- added SOT-23-3: SOT-23-3, digikey-footprints:SOT-23-3, F.Cu at (222.8, 72.1)
- added SOT-23-5: SOT-23-5, digikey-footprints:SOT-23-5, F.Cu at (213.9, 72.1)
- added TQFP-32 0.8 mm pitch: TQFP-32_7x7mm_Pitch0.8mm, Housings_QFP:TQFP-32_7x7mm_Pitch0.8mm, F.Cu at (195.1, 87.6)
Other:
- board text removed: "1 mil = 0.0254 mm"
